File: gpio_expansion.kicad_sch (KiCad schematic)
At the start: 4 parts, among them J8 EXPANSION_3V3, U1 STM32F446ZETx

Commit message: Publish corrected prototype package and documented engineering review
Changed lines of the file:
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@@
 		(comment 1 "Presentation refactor - hardware validation pending")
+	)
+	(rectangle
+		(start 275.59 157.734)
+		(end 276.606 157.734)
+		(stroke
+			(width 0)
+			(type default)
+		)
+		(fill
+			(type none)
+		)
 	)
 	(text "20-PIN EXPANSION HEADER"
