File: stm32.kicad_pcb (KiCad board)
At the start: 4 copper layers, 80 x 70 mm, 68 parts, among them J1 SWD, J2 USB_C_Receptacle_USB2.0_16P, J3 I²C1, J4 SPI1, J5 UART2_3V3, J6 ANALOG_3V3, J7 GPIO_D, J8 EXPANSION_3V3, SW1 SW_Push_Open, SW2 SW_Push_Open, SW3 SW_Push_Open, U1 STM32F446ZETx, U2 USBLC6-2SC6, U3 TPS7A2533DRVR, U4 TPS22918DBVR, Y1 8MHz

Commit message: Organize schematic into functional sheets with verified pin mapping
Connections:
- net /ANALOG0 renamed ANALOG0
- net /ANALOG1 renamed ANALOG1
- net /I²C1_SCL renamed I²C1_SCL
- net /I²C1_SDA renamed I²C1_SDA
- net /NRST renamed NRST
- net /PD0 renamed PD0
- net /PD1 renamed PD1
- net /PD2 renamed PD2
- net /PD3 renamed PD3
- net /PD4 renamed PD4
- net /PD5 renamed PD5
- net /PD6 renamed PD6
- net /PD7 renamed PD7
- net /PE10 renamed PE10
- net /PE11 renamed PE11
- net /PE12 renamed PE12
- net /PE13 renamed PE13
- net /PE14 renamed PE14
- net /PE15 renamed PE15
- net /PE8 renamed PE8
- net /PE9 renamed PE9
- net /PF6 renamed PF6
- net /PF7 renamed PF7
- net /PF8 renamed PF8
- net /PF9 renamed PF9
- net /PG11 renamed PG11
- net /PG13 renamed PG13
- net /PG14 renamed PG14
- net /PG9 renamed PG9
- net /SPI1_CS renamed SPI1_CS
- net /SPI1_MISO renamed SPI1_MISO
- net /SPI1_MOSI renamed SPI1_MOSI
- net /SPI1_SCK renamed SPI1_SCK
- net /START_CT renamed START_CT
- net /UART2_RX renamed UART2_RX
- net /UART2_TX renamed UART2_TX
- net /USB_D_N renamed USB_D_N
- net /USB_D_P renamed USB_D_P
- net /USB_VBUS renamed USB_VBUS
- net /USB_VBUS_FUSED renamed Net-(D5-A)
- net /USB_VBUS_RAW renamed USB_VBUS_RAW
- net /VREG_3V3 renamed VREG_3V3
- net Net-(J1-Pin_2) renamed SWDIO
- net Net-(J1-Pin_4) renamed SWCLK
- net Net-(J2-CC1) renamed USB_CC1
- net Net-(J2-CC2) renamed USB_CC2
- net Net-(SW1-B) renamed BOOT0
- net Net-(SW3-A) renamed USER_BUTTON
- net Net-(U1-PA9) renamed USB_VBUS_SENSE
- net Net-(U1-PB2) renamed BOOT1
- net Net-(U1-PC6) renamed LED1_GPIO
- net Net-(U1-PC7) renamed LED2_GPIO
- net Net-(U1-PH0) renamed HSE_IN
- net Net-(U1-PH1) renamed HSE_OUT
- net Net-(U1-VCAP_1) renamed MCU_VCAP1
- net Net-(U1-VCAP_2) renamed MCU_VCAP2

Commit message: Publish corrected prototype package and documented engineering review
Parts:
- added C29: 1µF, Capacitor_SMD:C_0603_1608Metric, F.Cu at (158.6, 114.6)
- moved C1 0.47 mm to (156.6, 113.2)
- moved C25 0.40 mm to (154.8, 119.7)
Routing:
- net PF7: track 105.9 -> 102.0 mm
- net PF8: track 53.0 -> 49.3 mm
- net USB_D_N: track 72.8 -> 76.4 mm
- net PE8: track 86.0 -> 89.6 mm
- net PF9: track 43.5 -> 40.0 mm
- net USB_VBUS: track 71.9 -> 74.9 mm
- net PD7: track 79.4 -> 81.6 mm
- net GND: track 71.2 -> 72.8 mm, vias 57 -> 59
- net PD3: track 50.9 -> 49.5 mm
- net PD0: track 43.3 -> 41.9 mm
- net PD1: track 36.9 -> 38.3 mm
- net PD5: track 37.7 -> 36.3 mm
- net PD2: track 42.7 -> 41.4 mm
- net PF6: track 44.6 -> 45.6 mm
- net NRST: track 64.3 -> 65.2 mm
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