File: usb_debug_clock.kicad_sch (KiCad schematic)
At the start: 17 parts, among them J1 SWD, J2 USB_C_Receptacle_USB2.0_16P, SW1 SW_Push_Open, SW2 SW_Push_Open, U2 USBLC6-2SC6, Y1 8MHz

Commit message: Publish corrected prototype package and documented engineering review
Parts:
- J1: LCSC Part Number C5142872 -> C55629812; Manufacturer CST -> SHOU HAN; Manufacturer Part Number CS-1109-1x5 (11.6) -> SH-PZ254V-1x5P
Changed lines of the file:
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@@
 			)
 		)
-		(property "Manufacturer" "CST"
+		(property "Manufacturer" "SHOU HAN"
 			(at 365.76 160.02 0)
 			(hide yes)
@@
 			)
 		)
-		(property "Manufacturer Part Number" "CS-1109-1x5 (11.6)"
+		(property "Manufacturer Part Number" "SH-PZ254V-1x5P"
 			(at 365.76 160.02 0)
 			(hide yes)
@@
 			)
 		)
-		(property "LCSC Part Number" "C5142872"
+		(property "LCSC Part Number" "C55629812"
 			(at 365.76 160.02 0)
 			(hide yes)
